Commit message: test new sdf

File: urdf/iiwa_gripper.urdf (robot description, URDF)
Before this commit: robot iiwa_14, 9 links, 8 joints
Links:
- added link base_link_link, mass 0.05; collision mesh filename=package://demonstrator6_description/meshes/collision/COL_ba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 scale=1 1 1; visual mesh filename=package://demonstrator6_description/meshes/visual/VIS_base.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 scale=1 1 1
- added link gripper_left_link, mass 0.01; collision mesh filename=package://demonstrator6_description/meshes/collision/COL_gr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 scale=1 1 1; visual mesh filename=package://demonstrator6_description/meshes/visual/VIS_gripp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 scale=1 1 1
- added link gripper_right_link, mass 0.01; collision mesh filename=package://demonstrator6_description/meshes/collision/COL_gr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 scale=1 1 1; visual mesh filename=package://demonstrator6_description/meshes/visual/VIS_gripp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 scale=1 1 1
- added link iiwa_link_ee
- added link iiwa_link_ee_kuka
- added link iiwa_link_ee_kuka_mft_pneum
- link iiwa_link_0: geometry collision mesh filename=package://demonstrator6_description/meshes/iiwa14/collision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; visual mesh filename=package://demonstrator6_description/meshes/iiwa14/visual/li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
- link iiwa_link_1: geometry collision mesh filename=package://demonstrator6_description/meshes/iiwa14/collision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; visual mesh filename=package://demonstrator6_description/meshes/iiwa14/visual/li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
- link iiwa_link_2: geometry collision mesh filename=package://demonstrator6_description/meshes/iiwa14/collision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; visual mesh filename=package://demonstrator6_description/meshes/iiwa14/visual/li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
- link iiwa_link_3: geometry collision mesh filename=package://demonstrator6_description/meshes/iiwa14/collision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; visual mesh filename=package://demonstrator6_description/meshes/iiwa14/visual/li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
- link iiwa_link_4: geometry collision mesh filename=package://demonstrator6_description/meshes/iiwa14/collision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; visual mesh filename=package://demonstrator6_description/meshes/iiwa14/visual/li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
- link iiwa_link_5: geometry collision mesh filename=package://demonstrator6_description/meshes/iiwa14/collision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; visual mesh filename=package://demonstrator6_description/meshes/iiwa14/visual/li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
- link iiwa_link_6: geometry collision mesh filename=package://demonstrator6_description/meshes/iiwa14/collision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; visual mesh filename=package://demonstrator6_description/meshes/iiwa14/visual/li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
- link iiwa_link_7: geometry collision mesh filename=package://demonstrator6_description/meshes/iiwa14/collision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; visual mesh filename=package://demonstrator6_description/meshes/iiwa14/visual/li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
Joints:
- added joint base_link_joint: type fixed, parent iiwa_link_7, child base_link_link, origin xyz=0 0 0.071 rpy=1.5707963705062866 -0 -0, axis 0 0 1, limit lower=1.0 upper=1.0 effort=100.0 velocity=1.0
- added joint gripper_left_joint: type prismatic, parent base_link_link, child gripper_left_link, origin xyz=-0.0850000023841858 0.050000011920928955 0 rpy=1.5707963705062866 1.570796251296997 0, axis 0 1 0, limit lower=0.0 upper=0.0704 effort=100.0 velocity=1.0
- added joint gripper_right_joint: type prismatic, parent base_link_link, child gripper_right_link, origin xyz=0.0850000023841858 0.050000011920928955 0 rpy=1.5707963705062866 -1.570796251296997 0, axis 0 1 0, limit lower=0.0 upper=0.0704 effort=100.0 velocity=1.0
- added joint iiwa_joint_ee: type fixed, parent iiwa_link_7, child iiwa_link_ee, origin xyz=0 0 0.045 rpy=0 -1.57079632679 0
- added joint iiwa_joint_ee_kuka: type fixed, parent iiwa_link_7, child iiwa_link_ee_kuka, origin xyz=0 0 0.045 rpy=3.14159265359 3.14159265359 3.14159265359, axis 0 0 1
- added joint iiwa_joint_ee_kuka_mft_pneum: type fixed, parent iiwa_link_7, child iiwa_link_ee_kuka_mft_pneum, origin xyz=0 0 0.071 rpy=0 -1.57079632679 0
- joint iiwa_joint_7: origin xyz=0 0.181 0 rpy=-1.57079632679 3.14159265359 0 -> xyz=0 0.081 0 rpy=-1.57079632679 3.14159265359 0
- joint world_iiwa_joint: origin xyz=0 0 0 rpy=0 0 0 -> xyz=0 0 0.0 rpy=0 0 0

Commit message: update urdf and sdf

File: urdf/iiwa_gripper.urdf (robot description, URDF)
Before this commit: robot iiwa14, 15 links, 14 joints
Links:
- removed link iiwa_link_ee
- removed link iiwa_link_ee_kuka
- removed link iiwa_link_ee_kuka_mft_pneum
- link iiwa_link_0: geometry collision mesh filename=package://demonstrator6_description/meshes/collision/link_0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; visual mesh filename=package://demonstrator6_description/meshes/visual/link_0.dae
- link iiwa_link_1: geometry collision mesh filename=package://demonstrator6_description/meshes/collision/link_1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; visual mesh filename=package://demonstrator6_description/meshes/visual/link_1.dae
- link iiwa_link_2: geometry collision mesh filename=package://demonstrator6_description/meshes/collision/link_2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; visual mesh filename=package://demonstrator6_description/meshes/visual/link_2.dae
- link iiwa_link_3: geometry collision mesh filename=package://demonstrator6_description/meshes/collision/link_3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; visual mesh filename=package://demonstrator6_description/meshes/visual/link_3.dae
- link iiwa_link_4: geometry collision mesh filename=package://demonstrator6_description/meshes/collision/link_4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; visual mesh filename=package://demonstrator6_description/meshes/visual/link_4.dae
- link iiwa_link_5: geometry collision mesh filename=package://demonstrator6_description/meshes/collision/link_5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; visual mesh filename=package://demonstrator6_description/meshes/visual/link_5.dae
- link iiwa_link_6: geometry collision mesh filename=package://demonstrator6_description/meshes/collision/link_6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; visual mesh filename=package://demonstrator6_description/meshes/visual/link_6.dae
- link iiwa_link_7: geometry collision mesh filename=package://demonstrator6_description/meshes/collision/link_7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; visual mesh filename=package://demonstrator6_description/meshes/visual/link_7.dae
Joints:
- removed joint iiwa_joint_ee
- removed joint iiwa_joint_ee_kuka
- removed joint iiwa_joint_ee_kuka_mft_pneum
- joint base_link_joint: origin xyz=0 0 0.071 rpy=1.5707963705062866 -0 -0 -> xyz=0 0 0.045 rpy=1.5707963705062866 -0 -0
